File: kicad-files/bitboy.kicad_pcb (KiCad board)
At the start: 2 copper layers, 58.3 x 50.3 mm, 7 parts, among them U1 XIAO-RP2040-DIP, U2 DM-OLED096-636, U3 ICM-42688-P

Commit message: Add screenshots
Parts:
- added G***: LOGO, LOGO, F.Cu at (130.1, 67.8)
- added G***: LOGO, LOGO, F.Cu at (146.3, 51.1)
- added G***: LOGO, LOGO, F.Cu at (171.1, 67.9)
- added G***: LOGO, LOGO, F.Cu at (123.7, 46.6)
- added G***: LOGO, LOGO, F.Cu at (169.1, 52.2)
- moved S1 1.10 mm to (168.2, 75.8)
Routing:
- net AddPeep: track 51.6 -> 50.6 mm
- net GND: track 63.7 -> 64.8 mm
Other:
- outline, holes or cut-outs redrawn
- board text added: "Reset"
- board text added: "Spawn More!"
